File: canosplit.kicad_sch (KiCad schematic)
At the start: 8 parts, among them J1 In, J2 Out, J3 Branch, J4 Power in

Commit message: researched parts
Parts:
- J1, J2, J3: footprint Connector_Molex:Molex_PicoBlade_53398-0471_1x04-1MP_P1.25mm_Vertical -> Connector_Molex:Molex_PicoBlade_53047-0410_1x04_P1.25mm_Vertical; Farnell_NO (none) -> 9733060
- J4: footprint Connector_Molex:Molex_PicoBlade_53398-0271_1x02-1MP_P1.25mm_Vertical -> Connector_Molex:Molex_PicoBlade_53047-0210_1x02_P1.25mm_Vertical; Farnell_NO (none) -> 9733051
- JP1, JP2, R1, R2: Farnell_NO (none) -> DO NOT ORDER
Changed lines of the file:
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@@
 (kicad_sch (version 20210621) (generator eeschema)
   (paper "A4")
-  (junction (at 106.68 82.55) (diameter 0) (color 0 0 0 0))
-  (junction (at 173.99 69.85) (diameter 0) (color 0 0 0 0))
-  (junction (at 106.68 105.41) (diameter 0) (color 0 0 0 0))
+  (junction (at 111.76 77.47) (diameter 0) (color 0 0 0 0))
   (junction (at 114.3 74.93) (diameter 0) (color 0 0 0 0))
   (junction (at 181.61 57.15) (diameter 0) (color 0 0 0 0))
   (junction (at 109.22 80.01) (diameter 0) (color 0 0 0 0))
-  (junction (at 111.76 77.47) (diameter 0) (color 0 0 0 0))
+  (junction (at 106.68 82.55) (diameter 0) (color 0 0 0 0))
+  (junction (at 106.68 105.41) (diameter 0) (color 0 0 0 0))
+  (junction (at 173.99 69.85) (diameter 0) (color 0 0 0 0))
   (wire (pts (xy 185.42 57.15) (xy 185.42 59.69))
     (stroke (width 0) (type default) (color 0 0 0 0))
@@
     (stroke (width 0) (type default) (color 0 0 0 0))
   )
+  (wire (pts (xy 130.81 105.41) (xy 106.68 105.41))
+    (stroke (width 0) (type default) (color 0 0 0 0))
+  )
   (wire (pts (xy 106.68 105.41) (xy 106.68 82.55))
     (stroke (width 0) (type default) (color 0 0 0 0))
   )
-  (wire (pts (xy 130.81 105.41) (xy 106.68 105.41))
-    (stroke (width 0) (type default) (color 0 0 0 0))
-  )
   (wire (pts (xy 87.63 80.01) (xy 109.22 80.01))
     (stroke (width 0) (type default) (color 0 0 0 0))
@@
     (stroke (width 0) (type default) (color 0 0 0 0))
   )
+  (wire (pts (xy 106.68 82.55) (xy 130.81 82.55))
+    (stroke (width 0) (type default) (color 0 0 0 0))
+  )
   (wire (pts (xy 87.63 82.55) (xy 106.68 82.55))
     (stroke (width 0) (type default) (color 0 0 0 0))
   )
-  (wire (pts (xy 106.68 82.55) (xy 130.81 82.55))
-    (stroke (width 0) (type default) (color 0 0 0 0))
-  )
   (wire (pts (xy 135.89 87.63) (xy 135.89 88.9))
     (stroke (width 0) (type default) (color 0 0 0 0))
@@
     (stroke (width 0) (type default) (color 0 0 0 0))
   )
+  (wire (pts (xy 114.3 97.79) (xy 114.3 74.93))
+    (stroke (width 0) (type default) (color 0 0 0 0))
+  )
   (wire (pts (xy 130.81 97.79) (xy 114.3 97.79))
-    (stroke (width 0) (type default) (color 0 0 0 0))
-  )
-  (wire (pts (xy 114.3 97.79) (xy 114.3 74.93))
     (stroke (width 0) (type default) (color 0 0 0 0))
   )
@@
       (effects (font (size 1.27 1.27)) hide)
     )
+    (property "Farnell_NO" "DO NOT ORDER" (id 4) (at 199.39 100.33 0)
+      (effects (font (size 1.27 1.27)) hide)
+    )
     (pin "1")
     (pin "2")
@@
     )
     (property "Datasheet" "~" (id 3) (at 199.39 110.49 0)
+      (effects (font (size 1.27 1.27)) hide)
+    )
+    (property "Farnell_NO" "DO NOT ORDER" (id 4) (at 199.39 110.49 0)
       (effects (font (size 1.27 1.27)) hide)
     )
@@
       (effects (font (size 1.27 1.27)) hide)
     )
+    (property "Farnell_NO" "DO NOT ORDER" (id 4) (at 170.18 110.49 0)
+      (effects (font (size 1.27 1.27)) hide)
+    )
     (pin "1")
     (pin "2")
@@
       (effects (font (size 1.27 1.27)) (justify left))
     )
-    (property "Footprint" "Connector_Molex:Molex_PicoBlade_53398-0271_1x02-1MP_P1.25mm_Vertical" (id 2) (at 181.61 72.39 0)
+    (property "Footprint" "Connector_Molex:Molex_PicoBlade_53047-0210_1x02_P1.25mm_Vertical" (id 2) (at 181.61 72.39 0)
       (effects (font (size 1.27 1.27)) hide)
     )
     (property "Datasheet" "~" (id 3) (at 181.61 72.39 0)
+      (effects (font (size 1.27 1.27)) hide)
+    )
+    (property "Farnell_NO" "9733051" (id 4) (at 181.61 72.39 0)
       (effects (font (size 1.27 1.27)) hide)
     )
@@
       (effects (font (size 1.27 1.27)) (justify left))
     )
-    (property "Footprint" "Connector_Molex:Molex_PicoBlade_53398-0471_1x04-1MP_P1.25mm_Vertical" (id 2) (at 135.89 77.47 0)
+    (property "Footprint" "Connector_Molex:Molex_PicoBlade_53047-0410_1x04_P1.25mm_Vertical" (id 2) (at 135.89 77.47 0)
       (effects (font (size 1.27 1.27)) hide)
     )
     (property "Datasheet" "~" (id 3) (at 135.89 77.47 0)
+      (effects (font (size 1.27 1.27)) hide)
+    )
+    (property "Farnell_NO" "9733060" (id 4) (at 135.89 77.47 0)
       (effects (font (size 1.27 1.27)) hide)
     )
@@
       (effects (font (size 1.27 1.27)) hide)
     )
+    (property "Farnell_NO" "DO NOT ORDER" (id 4) (at 170.18 100.33 0)
+      (effects (font (size 1.27 1.27)) hide)
+    )
     (pin "1")
     (pin "2")
@@
       (effects (font (size 1.27 1.27)) (justify left))
     )
-    (property "Footprint" "Connector_Molex:Molex_PicoBlade_53398-0471_1x04-1MP_P1.25mm_Vertical" (id 2) (at 135.89 100.33 0)
+    (property "Footprint" "Connector_Molex:Molex_PicoBlade_53047-0410_1x04_P1.25mm_Vertical" (id 2) (at 135.89 100.33 0)
       (effects (font (size 1.27 1.27)) hide)
     )
     (property "Datasheet" "~" (id 3) (at 135.89 100.33 0)
+      (effects (font (size 1.27 1.27)) hide)
+    )
+    (property "Farnell_NO" "9733060" (id 4) (at 135.89 100.33 0)
       (effects (font (size 1.27 1.27)) hide)
     )
@@
     (property "Reference" "J1" (id 0) (at 84.3915 68.58 0))
     (property "Value" "In" (id 1) (at 84.3915 71.12 0))
-    (property "Footprint" "Connector_Molex:Molex_PicoBlade_53398-0471_1x04-1MP_P1.25mm_Vertical" (id 2) (at 82.55 77.47 0)
+    (property "Footprint" "Connector_Molex:Molex_PicoBlade_53047-0410_1x04_P1.25mm_Vertical" (id 2) (at 82.55 77.47 0)
       (effects (font (size 1.27 1.27)) hide)
     )
     (property "Datasheet" "~" (id 3) (at 82.55 77.47 0)
+      (effects (font (size 1.27 1.27)) hide)
+    )
+    (property "Farnell_NO" "9733060" (id 4) (at 82.55 77.47 0)
       (effects (font (size 1.27 1.27)) hide)
     )
@@
     )
     (path "/f99dcfa0-a5e0-406d-a3d9-50dfad4eafa2"
-      (reference "J1") (unit 1) (value "In") (footprint "Connector_Molex:Molex_PicoBlade_53398-0471_1x04-1MP_P1.25mm_Vertical")
+      (reference "J1") (unit 1) (value "In") (footprint "Connector_Molex:Molex_PicoBlade_53047-0410_1x04_P1.25mm_Vertical")
     )
     (path "/85d1001a-4695-4d73-b936-3545a19383c1"
-      (reference "J2") (unit 1) (value "Out") (footprint "Connector_Molex:Molex_PicoBlade_53398-0471_1x04-1MP_P1.25mm_Vertical")
+      (reference "J2") (unit 1) (value "Out") (footprint "Connector_Molex:Molex_PicoBlade_53047-0410_1x04_P1.25mm_Vertical")
     )
     (path "/af01579c-856f-4a33-b635-4f3314f4a570"
-      (reference "J3") (unit 1) (value "Branch") (footprint "Connector_Molex:Molex_PicoBlade_53398-0471_1x04-1MP_P1.25mm_Vertical")
+      (reference "J3") (unit 1) (value "Branch") (footprint "Connector_Molex:Molex_PicoBlade_53047-0410_1x04_P1.25mm_Vertical")
     )
     (path "/64044cc6-c57d-4745-bd3d-83e0e2becef3"
-      (reference "J4") (unit 1) (value "Power in") (footprint "Connector_Molex:Molex_PicoBlade_53398-0271_1x02-1MP_P1.25mm_Vertical")
+      (reference "J4") (unit 1) (value "Power in") (footprint "Connector_Molex:Molex_PicoBlade_53047-0210_1x02_P1.25mm_Vertical")
     )
     (path "/a02cb009-ddf6-4c66-982d-59d9c190418c"

Commit message: updated after meeting
Parts:
- removed JP2: Termination, Jumper:SolderJumper-2_P1.3mm_Open_TrianglePad1.0x1.5mm, symbol Jumper:Jumper_2_Open
- removed R2: 120R, Resistor_SMD:R_0805_2012Metric, symbol Device:R
- JP1: footprint Jumper:SolderJumper-2_P1.3mm_Open_TrianglePad1.0x1.5mm -> Connector_PinHeader_2.54mm:PinHeader_1x03_P2.54mm_Vertical
Changed lines of the file:
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@@
   (paper "A4")
   (junction (at 111.76 77.47) (diameter 0) (color 0 0 0 0))
+  (junction (at 106.68 82.55) (diameter 0) (color 0 0 0 0))
+  (junction (at 181.61 57.15) (diameter 0) (color 0 0 0 0))
+  (junction (at 106.68 105.41) (diameter 0) (color 0 0 0 0))
+  (junction (at 109.22 80.01) (diameter 0) (color 0 0 0 0))
   (junction (at 114.3 74.93) (diameter 0) (color 0 0 0 0))
-  (junction (at 181.61 57.15) (diameter 0) (color 0 0 0 0))
-  (junction (at 109.22 80.01) (diameter 0) (color 0 0 0 0))
-  (junction (at 106.68 82.55) (diameter 0) (color 0 0 0 0))
-  (junction (at 106.68 105.41) (diameter 0) (color 0 0 0 0))
   (junction (at 173.99 69.85) (diameter 0) (color 0 0 0 0))
   (wire (pts (xy 185.42 57.15) (xy 185.42 59.69))
@@
     (stroke (width 0) (type default) (color 0 0 0 0))
   )
-  (wire (pts (xy 199.39 105.41) (xy 199.39 106.68))
-    (stroke (width 0) (type default) (color 0 0 0 0))
-  )
   (wire (pts (xy 114.3 68.58) (xy 114.3 74.93))
     (stroke (width 0) (type default) (color 0 0 0 0))
   )
-  (wire (pts (xy 199.39 92.71) (xy 212.09 92.71))
-    (stroke (width 0) (type default) (color 0 0 0 0))
-  )
   (wire (pts (xy 114.3 68.58) (xy 116.84 68.58))
     (stroke (width 0) (type default) (color 0 0 0 0))
@@
     (stroke (width 0) (type default) (color 0 0 0 0))
   )
-  (wire (pts (xy 199.39 114.3) (xy 199.39 115.57))
-    (stroke (width 0) (type default) (color 0 0 0 0))
-  )
   (wire (pts (xy 87.63 77.47) (xy 111.76 77.47))
     (stroke (width 0) (type default) (color 0 0 0 0))
@@
     (stroke (width 0) (type default) (color 0 0 0 0))
   )
+  (wire (pts (xy 171.45 72.39) (xy 176.53 72.39))
+    (stroke (width 0) (type default) (color 0 0 0 0))
+  )
   (wire (pts (xy 171.45 77.47) (xy 171.45 72.39))
     (stroke (width 0) (type default) (color 0 0 0 0))
   )
-  (wire (pts (xy 171.45 72.39) (xy 176.53 72.39))
-    (stroke (width 0) (type default) (color 0 0 0 0))
-  )
   (wire (pts (xy 173.99 69.85) (xy 176.53 69.85))
     (stroke (width 0) (type default) (color 0 0 0 0))
@@
     (stroke (width 0) (type default) (color 0 0 0 0))
   )
-  (wire (pts (xy 199.39 95.25) (xy 199.39 92.71))
-    (stroke (width 0) (type default) (color 0 0 0 0))
-  )
   (wire (pts (xy 181.61 55.88) (xy 181.61 57.15))
     (stroke (width 0) (type default) (color 0 0 0 0))
@@
     (stroke (width 0) (type default) (color 0 0 0 0))
   )
-  (wire (pts (xy 199.39 115.57) (xy 212.09 115.57))
-    (stroke (width 0) (type default) (color 0 0 0 0))
-  )
   (wire (pts (xy 114.3 97.79) (xy 114.3 74.93))
     (stroke (width 0) (type default) (color 0 0 0 0))
@@
   (wire (pts (xy 111.76 100.33) (xy 111.76 77.47))
     (stroke (width 0) (type default) (color 0 0 0 0))
-  )
-  (label "CAN_H" (at 212.09 92.71 0)
-    (effects (font (size 1.27 1.27)) (justify left bottom))
-  )
-  (label "CAN_L" (at 212.09 115.57 0)
-    (effects (font (size 1.27 1.27)) (justify left bottom))
   )
   (label "CAN_L" (at 182.88 115.57 0)
@@
   (label "CAN_H" (at 119.38 80.01 0)
     (effects (font (size 1.27 1.27)) (justify left bottom))
-  )
-  (symbol (lib_id "Jumper:Jumper_2_Open") (at 199.39 100.33 270) (unit 1)
-    (in_bom yes) (on_board yes) (fields_autoplaced)
-    (property "Reference" "JP2" (id 0) (at 201.93 99.0599 90)
-      (effects (font (size 1.27 1.27)) (justify left))
-    )
-    (property "Value" "Termination" (id 1) (at 201.93 101.5999 90)
-      (effects (font (size 1.27 1.27)) (justify left))
-    )
-    (property "Footprint" "Jumper:SolderJumper-2_P1.3mm_Open_TrianglePad1.0x1.5mm" (id 2) (at 199.39 100.33 0)
-      (effects (font (size 1.27 1.27)) hide)
-    )
-    (property "Datasheet" "~" (id 3) (at 199.39 100.33 0)
-      (effects (font (size 1.27 1.27)) hide)
-    )
-    (property "Farnell_NO" "DO NOT ORDER" (id 4) (at 199.39 100.33 0)
-      (effects (font (size 1.27 1.27)) hide)
-    )
-    (pin "1")
-    (pin "2")
-  )
-  (symbol (lib_id "Device:R") (at 199.39 110.49 0) (unit 1)
-    (in_bom yes) (on_board yes) (fields_autoplaced)
-    (property "Reference" "R2" (id 0) (at 201.93 109.2199 0)
-      (effects (font (size 1.27 1.27)) (justify left))
-    )
-    (property "Value" "120R" (id 1) (at 201.93 111.7599 0)
-      (effects (font (size 1.27 1.27)) (justify left))
-    )
-    (property "Footprint" "Resistor_SMD:R_0805_2012Metric" (id 2) (at 197.612 110.49 90)
-      (effects (font (size 1.27 1.27)) hide)
-    )
-    (property "Datasheet" "~" (id 3) (at 199.39 110.49 0)
-      (effects (font (size 1.27 1.27)) hide)
-    )
-    (property "Farnell_NO" "DO NOT ORDER" (id 4) (at 199.39 110.49 0)
-      (effects (font (size 1.27 1.27)) hide)
-    )
-    (pin "1")
-    (pin "2")
   )
   (symbol (lib_id "power:GND") (at 116.84 69.85 0) (unit 1)
@@
       (effects (font (size 1.27 1.27)) (justify left))
     )
-    (property "Footprint" "Jumper:SolderJumper-2_P1.3mm_Open_TrianglePad1.0x1.5mm" (id 2) (at 170.18 100.33 0)
+    (property "Footprint" "Connector_PinHeader_2.54mm:PinHeader_1x03_P2.54mm_Vertical" (id 2) (at 170.18 100.33 0)
       (effects (font (size 1.27 1.27)) hide)
     )
@@
     )
     (path "/a02cb009-ddf6-4c66-982d-59d9c190418c"
-      (reference "JP1") (unit 1) (value "Termination") (footprint "Jumper:SolderJumper-2_P1.3mm_Open_TrianglePad1.0x1.5mm")
-    )
-    (path "/16b33b0c-df47-440e-ae6b-6655a19a7803"
-      (reference "JP2") (unit 1) (value "Termination") (footprint "Jumper:SolderJumper-2_P1.3mm_Open_TrianglePad1.0x1.5mm")
+      (reference "JP1") (unit 1) (value "Termination") (footprint "Connector_PinHeader_2.54mm:PinHeader_1x03_P2.54mm_Vertical")
     )
     (path "/496ddb4f-c54e-4e5a-b066-0f7053818330"
       (reference "R1") (unit 1) (value "120R") (footprint "Resistor_SMD:R_0805_2012Metric")
     )
-    (path "/1d530c18-30ce-4e59-9474-6a5272471951"
-      (reference "R2") (unit 1) (value "120R") (footprint "Resistor_SMD:R_0805_2012Metric")
-    )
-  )
+  )

Commit message: updated board with new connector
Parts:
- J1, J2, J3: footprint Connector_Molex:Molex_PicoBlade_53047-0410_1x04_P1.25mm_Vertical -> Connector_Molex:Molex_CLIK-Mate_502382-0470_1x04-1MP_P1.25mm_Vertical
Changed lines of the file:
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@@
 (kicad_sch (version 20210621) (generator eeschema)
   (paper "A4")
+  (junction (at 106.68 105.41) (diameter 0) (color 0 0 0 0))
   (junction (at 111.76 77.47) (diameter 0) (color 0 0 0 0))
+  (junction (at 173.99 69.85) (diameter 0) (color 0 0 0 0))
+  (junction (at 109.22 80.01) (diameter 0) (color 0 0 0 0))
+  (junction (at 181.61 57.15) (diameter 0) (color 0 0 0 0))
+  (junction (at 114.3 74.93) (diameter 0) (color 0 0 0 0))
   (junction (at 106.68 82.55) (diameter 0) (color 0 0 0 0))
-  (junction (at 181.61 57.15) (diameter 0) (color 0 0 0 0))
-  (junction (at 106.68 105.41) (diameter 0) (color 0 0 0 0))
-  (junction (at 109.22 80.01) (diameter 0) (color 0 0 0 0))
-  (junction (at 114.3 74.93) (diameter 0) (color 0 0 0 0))
-  (junction (at 173.99 69.85) (diameter 0) (color 0 0 0 0))
   (wire (pts (xy 185.42 57.15) (xy 185.42 59.69))
     (stroke (width 0) (type default) (color 0 0 0 0))
@@
       (effects (font (size 1.27 1.27)) (justify left))
     )
-    (property "Footprint" "Connector_Molex:Molex_PicoBlade_53047-0410_1x04_P1.25mm_Vertical" (id 2) (at 135.89 77.47 0)
+    (property "Footprint" "Connector_Molex:Molex_CLIK-Mate_502382-0470_1x04-1MP_P1.25mm_Vertical" (id 2) (at 135.89 77.47 0)
       (effects (font (size 1.27 1.27)) hide)
     )
@@
       (effects (font (size 1.27 1.27)) (justify left))
     )
-    (property "Footprint" "Connector_Molex:Molex_PicoBlade_53047-0410_1x04_P1.25mm_Vertical" (id 2) (at 135.89 100.33 0)
+    (property "Footprint" "Connector_Molex:Molex_CLIK-Mate_502382-0470_1x04-1MP_P1.25mm_Vertical" (id 2) (at 135.89 100.33 0)
       (effects (font (size 1.27 1.27)) hide)
     )
@@
     (property "Reference" "J1" (id 0) (at 84.3915 68.58 0))
     (property "Value" "In" (id 1) (at 84.3915 71.12 0))
-    (property "Footprint" "Connector_Molex:Molex_PicoBlade_53047-0410_1x04_P1.25mm_Vertical" (id 2) (at 82.55 77.47 0)
+    (property "Footprint" "Connector_Molex:Molex_CLIK-Mate_502382-0470_1x04-1MP_P1.25mm_Vertical" (id 2) (at 82.55 77.47 0)
       (effects (font (size 1.27 1.27)) hide)
     )
@@
     )
     (path "/f99dcfa0-a5e0-406d-a3d9-50dfad4eafa2"
-      (reference "J1") (unit 1) (value "In") (footprint "Connector_Molex:Molex_PicoBlade_53047-0410_1x04_P1.25mm_Vertical")
+      (reference "J1") (unit 1) (value "In") (footprint "Connector_Molex:Molex_CLIK-Mate_502382-0470_1x04-1MP_P1.25mm_Vertical")
     )
     (path "/85d1001a-4695-4d73-b936-3545a19383c1"
-      (reference "J2") (unit 1) (value "Out") (footprint "Connector_Molex:Molex_PicoBlade_53047-0410_1x04_P1.25mm_Vertical")
+      (reference "J2") (unit 1) (value "Out") (footprint "Connector_Molex:Molex_CLIK-Mate_502382-0470_1x04-1MP_P1.25mm_Vertical")
     )
     (path "/af01579c-856f-4a33-b635-4f3314f4a570"
-      (reference "J3") (unit 1) (value "Branch") (footprint "Connector_Molex:Molex_PicoBlade_53047-0410_1x04_P1.25mm_Vertical")
+      (reference "J3") (unit 1) (value "Branch") (footprint "Connector_Molex:Molex_CLIK-Mate_502382-0470_1x04-1MP_P1.25mm_Vertical")
     )
     (path "/64044cc6-c57d-4745-bd3d-83e0e2becef3"
